Commit message: Make the Onshape model drive and dig in Gazebo
Repair the raw Onshape export with scripts so it can be regenerated on
every re-export, and wire it up to ros2_control in Gazebo.

- fix_kinematics.py rebuilds the joint tree without moving any part:
  one wheel per flange with consistent axes, chassis frame fixed to root,
  excavator ladder on a prismatic lift with driven and idler rollers,
  loop-closure dummies and <mimic> couplings removed.
- Buckets ride three joints each so belt_animator.py can run them round
  the belt loop, slaved to the drive roller (Gazebo and RViz).
- Collision geometry generated from the meshes: boxes for extrusions,
  cylinders for wheels/rollers/shafts, meshes for buckets and the bin.
- add_ros2_control.py adds wheel, excavator and bucket hardware blocks,
  with buckets starting at their CAD poses.
- gazebo.launch.py expands $(find) for the controllers file, adds the
  mesh resource path, passes params to the spawners, spawns above ground.
- Controllers moved to ForwardCommandController (velocity_/position_
  controllers no longer exist in Lyrical).
- Old ROS 1 export moved to old_urdf/; README documents usage.

File: src/lunabotics_model/urdf/assembly_1.urdf (robot description, URDF)
Before this commit: robot assembly_1, 31 links, 30 joints
Links:
- added link 30___30___403_4, mass 0.518626; visual mesh filename=package://lunabotics_model/meshes/_30___30___403_1.stl scale=1 1 1
- added link 30___30___403_5, mass 0.518626; visual mesh filename=package://lunabotics_model/meshes/_30___30___403_1.stl scale=1 1 1
- added link 30___30___403__1__loop_closure, mass 1e-09
- added link 30___30___403__3__loop_closure, mass 1e-09
- added link 30___60___400_2, mass 0.875901; visual mesh filename=package://lunabotics_model/meshes/_30___60___400_1.stl scale=1 1 1
- added link 30___60___400_3, mass 0.875901; visual mesh filename=package://lunabotics_model/meshes/_30___60___400_1.stl scale=1 1 1
- added link 30___60___400__1__loop_closure, mass 1e-09
- added link 30___60___400__3__loop_closure, mass 1e-09
- added link belt, mass 0.638071; visual mesh filename=package://lunabotics_model/meshes/belt.stl scale=1 1 1
- added link bucket, mass 0.00222098; visual mesh filename=package://lunabotics_model/meshes/bucket.stl scale=1 1 1
- added link bucket_1, mass 0.148585; visual mesh filename=package://lunabotics_model/meshes/bucket_1.stl scale=1 1 1
- added link bucket_10, mass 0.148585; visual mesh filename=package://lunabotics_model/meshes/bucket_1.stl scale=1 1 1
- added link bucket_2, mass 0.148585; visual mesh filename=package://lunabotics_model/meshes/bucket_1.stl scale=1 1 1
- added link bucket_3, mass 0.148585; visual mesh filename=package://lunabotics_model/meshes/bucket_1.stl scale=1 1 1
- added link bucket_4, mass 0.148585; visual mesh filename=package://lunabotics_model/meshes/bucket_1.stl scale=1 1 1
- added link bucket_5, mass 0.148585; visual mesh filename=package://lunabotics_model/meshes/bucket_1.stl scale=1 1 1
- added link bucket_6, mass 0.148585; visual mesh filename=package://lunabotics_model/meshes/bucket_1.stl scale=1 1 1
- added link bucket_7, mass 0.148585; visual mesh filename=package://lunabotics_model/meshes/bucket_1.stl scale=1 1 1
- added link bucket_8, mass 0.148585; visual mesh filename=package://lunabotics_model/meshes/bucket_1.stl scale=1 1 1
- added link bucket_9, mass 0.148585; visual mesh filename=package://lunabotics_model/meshes/bucket_1.stl scale=1 1 1
- added link cylindrical_1
- added link cylindrical_1_1
- added link cylindrical_1_loop_closure
- added link electronics, mass 0.00143041; visual mesh filename=package://lunabotics_model/meshes/electronics.stl scale=1 1 1
- added link rod, mass 0.126439; visual mesh filename=package://lunabotics_model/meshes/rod.stl scale=1 1 1
- added link rod_1, mass 0.126439; visual mesh filename=package://lunabotics_model/meshes/rod.stl scale=1 1 1
- added link rod__2__loop_closure, mass 1e-09
- added link roller, mass 2.28767; visual mesh filename=package://lunabotics_model/meshes/roller.stl scale=1 1 1
- added link roller_1, mass 2.28767; visual mesh filename=package://lunabotics_model/meshes/roller.stl scale=1 1 1
- added link slider_bracket, mass 0.060264; visual mesh filename=package://lunabotics_model/meshes/slider_bracket.stl scale=1 1 1
- added link slider_bracket_1, mass 0.060264; visual mesh filename=package://lunabotics_model/meshes/slider_bracket.stl scale=1 1 1
- added link slider_bracket__2__loop_closure, mass 1e-09
- added link slider_bracket__5__loop_closure, mass 1e-09
- link root: geometry visual mesh filename=package://lunabotics_model/meshes/_57BLR50_24_01_P1_Back.stl scale=1 1 1; visual mesh filename=package://lunabotics_model/meshes/_57BLR50_24_01_P1_Back.stl scale=1 1 1
- link wheel: mass 8.93632 -> 9.11886
- link wheel_1: mass 8.93632 -> 9.11886
- link wheel_mirrored: mass 8.93631 -> 9.11886
- link wheel_mirrored_1: mass 8.93631 -> 9.11886
Joints:
- added joint cylindrical_1: type prismatic, parent roller, child cylindrical_1, origin xyz=-0.208047 0.615806 -5.27356e-15 rpy=-3.14159 1.6291e-15 -1.24499, axis -0 -0 1, limit lower=0 upper=0 effort=1 velocity=1, mimic joint=cylindrical_1_2 multiplier=1 offset=0
- added joint cylindrical_1_1: type continuous, parent cylindrical_1, child rod, origin xyz=0 0 0 rpy=0 -0 0, axis -0 -0 1, mimic joint=cylindrical_1_3 multiplier=-1 offset=0
- added joint cylindrical_1_2: type prismatic, parent roller, child cylindrical_1_1, origin xyz=7.77156e-16 -3.10862e-15 -1.95954e-14 rpy=3.14159 -3.71581e-14 1.8966, axis -0 -0 1, limit lower=0 upper=0 effort=1 velocity=1
- added joint cylindrical_1_3: type continuous, parent cylindrical_1_1, child rod_1, origin xyz=0 0 0 rpy=0 -0 0, axis -0 -0 1
- added joint cylindrical_1_loop_closure: type prismatic, parent roller_1, child cylindrical_1_loop_closure, origin xyz=0 0 -2.94209e-15 rpy=-3.14159 1.63186e-15 -1.24499, axis -0 -0 1, limit lower=0 upper=0 effort=1 velocity=1
- added joint cylindrical_1_loop_closure_1: type continuous, parent cylindrical_1_loop_closure, child rod__2__loop_closure, origin xyz=0 0 0 rpy=0 -0 0, axis -0 -0 1
- added joint fastened_16: type fixed, parent 30___60___400_3, child 30___30___403, origin xyz=0.0353602 0.0055 -2.77556e-17 rpy=1.5708 0.959931 3.14159, axis 0.573576 0.819152 -0
- added joint fastened_17: type fixed, parent 40___40___1_1, child bucket, origin xyz=-0.00387893 0.2 -0.01775 rpy=-3.14159 -1.15367e-16 4.16334e-17, axis 0 1 0
- added joint fastened_1_1: type fixed, parent rod, child 30___30___403_4, origin xyz=0.65 4.996e-16 0.1325 rpy=-1.80176e-16 3.53474e-14 -3.14159, axis -0 -0 -1
- added joint fastened_1_2: type fixed, parent bucket, child electronics, origin xyz=-0.128628 1.11022e-16 0.0958044 rpy=0 1.5708 3.78956e-17, axis -0.80193 0 0.597418
- added joint fastened_1_3: type fixed, parent 30___30___1, child 40___40___1, origin xyz=-0.402 -0.0153602 -0.015 rpy=-7.68143e-16 -3.18924e-15 -2.28983e-16, axis 0 1 0
- added joint fastened_1_loop_closure: type fixed, parent rod_1, child 30___30___403__3__loop_closure, origin xyz=2.93099e-14 5.55112e-16 -0.1325 rpy=3.14159 -1.50644e-14 -1.11022e-15, axis -0 -0 -1
- added joint fastened_1_loop_closure_1: type fixed, parent rod_1, child 30___30___403__1__loop_closure, origin xyz=1.11022e-16 -5.55112e-17 0.1325 rpy=-1.83143e-17 -2.72895e-17 -1.11022e-16, axis -0 -0 -1
- added joint fastened_2_1: type fixed, parent slider_bracket, child 30___60___400_3, origin xyz=-0.320525 -0.0275 -0.011 rpy=0 1.5708 1.5708, axis 0 -1 0
- added joint fastened_2_2: type fixed, parent 40___40___1, child 30___30___2, origin xyz=0.1835 -0.4097 0.001129 rpy=-8.18156e-17 -1.45482e-16 4.85722e-17, axis 0 1 0
- added joint fastened_2_loop_closure: type fixed, parent slider_bracket_1, child 30___60___400__3__loop_closure, origin xyz=-0.320525 0.0275 -0.011 rpy=0 1.5708 1.5708, axis 0 -1 0
- added joint fastened_2_loop_closure_1: type fixed, parent slider_bracket_1, child 30___60___400__1__loop_closure, origin xyz=0.034125 0.0275 -0.011 rpy=0 1.5708 -1.5708, axis 0 -1 0
- added joint fastened_3_1: type fixed, parent belt, child roller_1, origin xyz=0.0219432 0.086578 -1.78191e-14 rpy=-2.88933e-14 -1.49374e-14 -9.71445e-16, axis -0 -0 1
- added joint fastened_4_1: type fixed, parent belt, child roller, origin xyz=0.22999 -0.529228 4.16334e-15 rpy=-2.8894e-14 -1.495e-14 -1.11022e-15, axis -0 -0 1
- added joint fastened_5_1: type fixed, parent belt, child bucket_6, origin xyz=0.120027 -0.355272 1.27121e-14 rpy=3.14159 1.95116e-14 -2.48998, axis -0.947393 -0.320072 -9.88829e-15
- added joint fastened_5_2: type fixed, parent belt, child bucket_9, origin xyz=0.080018 -0.236848 8.43769e-15 rpy=3.14159 1.95116e-14 -2.48998, axis -0.947393 -0.320072 -9.88829e-15
- added joint fastened_5_3: type fixed, parent belt, child bucket_3, origin xyz=0 1.38778e-16 0 rpy=3.14159 1.94584e-14 -2.48998, axis -0.947393 -0.320072 -9.88829e-15
- added joint fastened_5_4: type fixed, parent bucket_1, child belt, origin xyz=-0.0980839 0.44185 -0.165 rpy=3.14159 1.78598e-14 -2.48998, axis -0.947393 -0.320072 -9.88829e-15
- added joint fastened_5_5: type fixed, parent 30___30___1, child 30___30___403_3, origin xyz=-0.437 0 -1.66533e-16 rpy=0 -1.5708 -1.5708, axis -1 0 0
- added joint fastened_6_1: type fixed, parent belt, child bucket_10, origin xyz=0.251933 -0.44265 1.78746e-14 rpy=3.14159 -1.99225e-14 0.651611, axis -0.947393 -0.320072 -9.88829e-15
- added joint fastened_6_2: type fixed, parent belt, child bucket_7, origin xyz=0.211924 -0.324225 1.37113e-14 rpy=3.14159 -1.99225e-14 0.651611, axis -0.947393 -0.320072 -9.88829e-15
- added joint fastened_6_3: type fixed, parent belt, child bucket_5, origin xyz=0.171915 -0.205801 9.4369e-15 rpy=3.14159 -1.99225e-14 0.651611, axis -0.947393 -0.320072 -9.88829e-15
- added joint fastened_6_4: type fixed, parent belt, child bucket_2, origin xyz=0.0918971 0.031047 9.4369e-16 rpy=3.14159 -1.97799e-14 0.651611, axis -0.947393 -0.320072 -9.88829e-15
- added joint fastened_6_5: type fixed, parent 30___30___403, child 30___30___1, origin xyz=0.2015 -0.1042 -0.398 rpy=-1.5708 -5.55112e-16 1.5708, axis -0 -0 1
- added joint slider_1: type prismatic, parent 30___30___403_5, child slider_bracket, origin xyz=0.374783 0.015 0.0107 rpy=0 -1.5708 -4.71239, axis -0 -1 -0, limit lower=-10000 upper=10000 effort=1 velocity=1, mimic joint=slider_1_1 multiplier=1 offset=0
- added joint slider_1_1: type prismatic, parent 30___30___403_5, child slider_bracket_1, origin xyz=0.374783 0.015 -0.2757 rpy=0 1.5708 -1.5708, axis -0 -1 -0, limit lower=-10000 upper=10000 effort=1 velocity=1
- added joint slider_1_loop_closure: type prismatic, parent 30___30___403_4, child slider_bracket__5__loop_closure, origin xyz=0.374783 -0.015 -0.2757 rpy=0 1.5708 1.5708, axis -0 -1 -0, limit lower=-10000 upper=10000 effort=1 velocity=1, mimic joint=slider_1_1 multiplier=1 offset=0
- added joint slider_1_loop_closure_1: type prismatic, parent 30___30___403_4, child slider_bracket__2__loop_closure, origin xyz=0.374783 -0.015 0.0107 rpy=0 -1.5708 4.71239, axis -0 -1 -0, limit lower=-10000 upper=10000 effort=1 velocity=1
- joint fastened_1: axis 0 1 0 -> -0 -0 -1; child 40___40___1 -> 30___30___403_5; origin xyz=0.035 -0.0153602 -0.015 rpy=-7.68143e-16 -3.18924e-15 -2.28983e-16 -> xyz=0.65 -1.11022e-16 -0.1325 rpy=3.14159 2.03102e-14 -3.14159; parent 30___30___1 -> rod
- joint fastened_10: origin xyz=-0.226225 -0.0178602 0 rpy=1.5708 -2.3707e-17 -1.52834e-16 -> xyz=-0.024725 -0.12206 -0.398 rpy=1.5708 -2.3707e-17 -1.52834e-16
- joint fastened_11: origin xyz=0.0443602 -0.563 0.015 rpy=-3.14159 5.10127e-16 1.5708 -> xyz=-0.00536018 0.015 0.015 rpy=-3.14159 5.10127e-16 1.5708
- joint fastened_12: origin xyz=0.0443602 0.015 0.015 rpy=-3.14159 1.29557e-15 1.5708 -> xyz=-0.00536018 0.593 0.015 rpy=-3.14159 1.29557e-15 1.5708
- joint fastened_13: origin xyz=0.0153602 -0.22 0.0055 rpy=-6.9456e-17 -2.62025e-16 -1.5708 -> xyz=0.0153602 -0.3 0.0055 rpy=6.61744e-24 -7.34684e-40 -1.5708
- joint fastened_14: child 57blr70_24_02_hg50_p5_2 -> 57blr70_24_02_hg50_p5__1_; origin xyz=2.77556e-16 -0.55 5.55112e-17 rpy=-3.14159 7.73892e-16 1.5708 -> xyz=0.0951728 0.120338 -0.0606898 rpy=-1.5708 -1.48353 -1.5708
- joint fastened_14_1: child 57blr70_24_02_hg50_p5__1__1 -> 57blr70_24_02_hg50_p5_2; origin xyz=0.144893 -0.457662 -0.0606898 rpy=-1.5708 -1.48353 -1.5708 -> xyz=-0.0497204 0.028 6.245e-17 rpy=-3.14159 7.73892e-16 1.5708
- joint fastened_14_2: child 57blr70_24_02_hg50_p5_3 -> 57blr70_24_02_hg50_p5__1__1; origin xyz=5.55112e-17 1.11022e-16 -2.08167e-17 rpy=-3.14159 1.7604e-15 1.5708 -> xyz=0.0951728 0.120338 -0.0606898 rpy=-1.5708 -1.48353 -1.5708
- joint fastened_14_3: axis -2.22045e-16 -0 1 -> 0 0 1; child 30___30___700_1 -> 57blr70_24_02_hg50_p5_3; origin xyz=0.020571 -0.46121 -0.127393 rpy=0 -1.5708 3.05433 -> xyz=-0.0497204 0.578 -1.38778e-17 rpy=-3.14159 1.7604e-15 1.5708; parent 57blr70_24_02_hg50_p5__1_ -> 30___30___700_1
- joint fastened_15: origin xyz=-0.497574 -0.52582 -0.234351 rpy=3.11379e-15 -3.46945e-15 -1.19665e-15 -> xyz=0.535533 -0.52582 -0.125315 rpy=-7.86541e-16 4.14946e-15 1.48463e-15
- joint fastened_15_1: origin xyz=-1.66533e-16 -0.52582 -1.66533e-16 rpy=2.01041e-15 -2.9976e-15 -6.02292e-16 -> xyz=-1.11022e-16 -0.52582 1.00614e-16 rpy=5.46607e-16 -4.16334e-17 -1.07669e-15
- joint fastened_15_2: origin xyz=-0.497574 0.027 -0.234351 rpy=3.14159 -3.38618e-15 -1.26378e-15 -> xyz=0.535533 0.027 -0.125315 rpy=3.14159 2.83107e-15 -4.6597e-16
- joint fastened_15_3: origin xyz=1.11022e-16 0.027 0 rpy=-3.14159 2.77556e-17 -1.95372e-16 -> xyz=-4.996e-16 0.027 -2.18575e-16 rpy=3.14159 3.08087e-15 -8.03265e-16
- joint fastened_2: axis 0 1 0 -> 0 -1 0; child 30___30___2 -> 30___60___400_2; origin xyz=0.1835 -0.4097 0.001129 rpy=-8.18156e-17 -1.45482e-16 4.85722e-17 -> xyz=0.034125 -0.0275 -0.011 rpy=0 1.5708 -1.5708; parent 40___40___1 -> slider_bracket
- joint fastened_5: axis -0 -0 1 -> -0.947393 -0.320072 -9.88829e-15; child 30___30___1 -> bucket_8; origin xyz=-0.4125 0.015 -1.38778e-17 rpy=1.5708 8.32667e-16 1.5708 -> xyz=0.160036 -0.473697 1.68754e-14 rpy=3.14159 1.95116e-14 -2.48998; parent 30___30___403_3 -> belt
- joint fastened_6: axis 1 0 0 -> -0.947393 -0.320072 -9.88829e-15; child 30___30___403 -> bucket_4; origin xyz=0.437 0 0 rpy=0 1.5708 -1.5708 -> xyz=0.131906 -0.0873772 5.21805e-15 rpy=3.14159 -1.98757e-14 0.651611; parent 30___30___1 -> belt
- joint fastened_7: axis 1 -0 -0 -> 1 0 0; child 30___30___403_3 -> 30___30___700_1; origin xyz=0.0497204 -0.578 6.93889e-18 rpy=-3.14159 4.57243e-16 -3.14159 -> xyz=0.4125 -0.015 0 rpy=-3.14159 -4.57243e-16 -3.14159; parent 30___30___700_1 -> 30___30___403_3
- joint hanging_node_to_root_joint: child 57blr70_24_02_hg50_p5__1_ -> bucket_1; origin xyz=0 0 0 rpy=0 -0 0 -> xyz=0.382957 -0.681137 -0.0586148 rpy=1.5708 0.936671 1.48353
- joint revolute_1: origin xyz=-0.55 -5.55112e-17 0.0167 rpy=1.5708 -2.19269e-15 0.44017 -> xyz=-0.55 3.05311e-16 0.0167 rpy=1.5708 -3.89966e-15 2.91173
- joint revolute_1_1: origin xyz=-0.55 -1.38778e-16 -0.48212 rpy=-1.5708 -5.55112e-17 -2.70142 -> xyz=-0.55 2.498e-16 -0.48212 rpy=-1.5708 3.33067e-16 -0.229865
- joint revolute_1_2: origin xyz=1.11022e-16 -2.77556e-17 -0.48212 rpy=-1.5708 -1.60982e-15 -2.70142 -> xyz=-4.996e-16 3.60822e-16 -0.48212 rpy=-1.5708 4.85723e-16 -0.229865
- joint revolute_1_3: origin xyz=-1.11022e-16 -8.32667e-17 0.0167 rpy=1.5708 9.15934e-16 0.44017 -> xyz=-3.88578e-16 2.77556e-16 0.0167 rpy=1.5708 6.93889e-16 2.91173
