Commit message: Add base_link frame and MuJoCo bucket digging test
- fix_kinematics.py adds base_link as the tree root (x forward, y left,
  z up, origin on the ground between the wheels); the Onshape root sat
  5 deg off the chassis. diff_drive_controller, spawn height and docs
  updated to match.
- mujoco_dig/dig_test.py: MuJoCo scene built from the repaired URDF with
  the CAD buckets and bin (split into convex wall slabs), the full robot
  as visuals, and a regolith pit; runs the belt and counts particles
  lifted and delivered to the bin.
- README and guide updated.

File: src/lunabotics_model/urdf/assembly_1_fixed.urdf (robot description, URDF)
Before this commit: robot assembly_1, 74 links, 73 joints
Links:
- added link base_link
Joints:
- added joint base_link_to_root: type fixed, parent base_link, child root, origin xyz=-0.182662687 -0.275898208 0.307894177 rpy=0 -0 1.65805916

File: src/lunabotics_model/urdf/assembly_1_sim.urdf (robot description, URDF)
Before this commit: robot assembly_1, 74 links, 73 joints
Links:
- added link base_link
Joints:
- added joint base_link_to_root: type fixed, parent base_link, child root, origin xyz=-0.182662687 -0.275898208 0.307894177 rpy=0 -0 1.65805916

Commit message: Add Artemis Arena with BP-1, real robot mass and drive motor limits
- generate_arena_world.py writes the Lunabotics Artemis Arena (6.88 x 5 m,
  guidebook layout or random --seed): BP-1 floor mesh with craters and
  gravel roughness, rocks, column, walls and zone outlines.
  world:=artemis_arena spawns the robot in the starting zone; x/y/yaw
  launch arguments override the spawn pose.
- fix_kinematics.py rebuilds masses to the measured 50 kg (datasheet
  gearmotor masses, CAD frame/excavator, stated assumptions for battery
  and bin, wheels take the remainder) and limits the wheels to the
  57BLR70-24-02-HG50 gearmotor: 20 N*m, 70 rpm.
- README and guide updated.

File: src/lunabotics_model/urdf/assembly_1_fixed.urdf (robot description, URDF)
Before this commit: robot assembly_1, 75 links, 74 joints
Links:
- link bucket: mass 0.00222098 -> 1.5
- link electronics: mass 0.00143041 -> 5
- link root: mass None -> 5.96
- link wheel: mass 9.11886 -> 5.18587
- link wheel_1: mass 9.11886 -> 5.18587
- link wheel_mirrored: mass 9.11886 -> 5.18587
- link wheel_mirrored_1: mass 9.11886 -> 5.18587
Joints:
- joint revolute_1: limit (none) -> effort=20 velocity=7.33038286
- joint revolute_1_1: limit (none) -> effort=20 velocity=7.33038286
- joint revolute_1_2: limit (none) -> effort=20 velocity=7.33038286
- joint revolute_1_3: limit (none) -> effort=20 velocity=7.33038286

File: src/lunabotics_model/urdf/assembly_1_sim.urdf (robot description, URDF)
Before this commit: robot assembly_1, 75 links, 74 joints
Links:
- link bucket: mass 0.00222098 -> 1.5
- link electronics: mass 0.00143041 -> 5
- link root: mass None -> 5.96
- link wheel: mass 9.11886 -> 5.18587
- link wheel_1: mass 9.11886 -> 5.18587
- link wheel_mirrored: mass 9.11886 -> 5.18587
- link wheel_mirrored_1: mass 9.11886 -> 5.18587
Joints:
- joint revolute_1: limit (none) -> effort=20 velocity=7.33038286
- joint revolute_1_1: limit (none) -> effort=20 velocity=7.33038286
- joint revolute_1_2: limit (none) -> effort=20 velocity=7.33038286
- joint revolute_1_3: limit (none) -> effort=20 velocity=7.33038286

Commit message: Add wheel slip on the regolith (Gazebo WheelSlip)
- add_ros2_control.py adds the WheelSlip system to the four drive wheels:
  compliance 0.6 forward and sideways (estimate for loose sand), wheel
  load from the 50 kg mass. The robot now spins up gradually from rest
  and can pivot on the spot with the 20 N*m motors.
- fix_kinematics.py drops the flange collision (hidden in the hub);
  WheelSlip needs exactly one collision per wheel link.
- README and guide updated.

File: src/lunabotics_model/urdf/assembly_1_fixed.urdf (robot description, URDF)
Before this commit: robot assembly_1, 75 links, 74 joints
Links:
- link flange: geometry visual mesh filename=package://lunabotics_model/meshes/flange.stl scale=1 1 1
- link flange_1: geometry visual mesh filename=package://lunabotics_model/meshes/flange.stl scale=1 1 1
- link flange_2: geometry visual mesh filename=package://lunabotics_model/meshes/flange.stl scale=1 1 1
- link flange_3: geometry visual mesh filename=package://lunabotics_model/meshes/flange.stl scale=1 1 1

File: src/lunabotics_model/urdf/assembly_1_sim.urdf (robot description, URDF)
Before this commit: robot assembly_1, 75 links, 74 joints
Links:
- link flange: geometry visual mesh filename=package://lunabotics_model/meshes/flange.stl scale=1 1 1
- link flange_1: geometry visual mesh filename=package://lunabotics_model/meshes/flange.stl scale=1 1 1
- link flange_2: geometry visual mesh filename=package://lunabotics_model/meshes/flange.stl scale=1 1 1
- link flange_3: geometry visual mesh filename=package://lunabotics_model/meshes/flange.stl scale=1 1 1

Commit message: Belt drive roller limits from TSINY TS-30GZ6287-R-LS (6 N*m, 50 rpm)

File: src/lunabotics_model/urdf/assembly_1_fixed.urdf (robot description, URDF)
Before this commit: robot assembly_1, 75 links, 74 joints
Joints:
- joint drive_roller_joint: limit effort=50 velocity=20 -> effort=6 velocity=5.23598776
- joint idler_roller_joint: limit effort=50 velocity=20 -> effort=6 velocity=5.23598776

File: src/lunabotics_model/urdf/assembly_1_sim.urdf (robot description, URDF)
Before this commit: robot assembly_1, 75 links, 74 joints
Joints:
- joint drive_roller_joint: limit effort=50 velocity=20 -> effort=6 velocity=5.23598776
- joint idler_roller_joint: limit effort=50 velocity=20 -> effort=6 velocity=5.23598776

File: src/lunabotics_model/urdf/assembly_1_sim_bekker.urdf (robot description, URDF)
Before this commit: robot assembly_1, 75 links, 74 joints
Joints:
- joint drive_roller_joint: limit effort=50 velocity=20 -> effort=6 velocity=5.23598776
- joint idler_roller_joint: limit effort=50 velocity=20 -> effort=6 velocity=5.23598776

Commit message: Excavator lift limits from the PA-14-6-35 linear actuator (156 N, 2 in/s, 6 in stroke)

File: src/lunabotics_model/urdf/assembly_1_fixed.urdf (robot description, URDF)
Before this commit: robot assembly_1, 75 links, 74 joints
Joints:
- joint excavator_lift: limit lower=-0.15 upper=0.15 effort=500 velocity=0.05 -> lower=-0.1524 upper=0 effort=155.68777 velocity=0.0508

File: src/lunabotics_model/urdf/assembly_1_sim.urdf (robot description, URDF)
Before this commit: robot assembly_1, 75 links, 74 joints
Joints:
- joint excavator_lift: limit lower=-0.15 upper=0.15 effort=500 velocity=0.05 -> lower=-0.1524 upper=0 effort=155.68777 velocity=0.0508

File: src/lunabotics_model/urdf/assembly_1_sim_bekker.urdf (robot description, URDF)
Before this commit: robot assembly_1, 75 links, 74 joints
Joints:
- joint excavator_lift: limit lower=-0.15 upper=0.15 effort=500 velocity=0.05 -> lower=-0.1524 upper=0 effort=155.68777 velocity=0.0508

Commit message: Excavator lift: two PA-14-6-35 actuators, one each side (311 N combined)

File: src/lunabotics_model/urdf/assembly_1_fixed.urdf (robot description, URDF)
Before this commit: robot assembly_1, 75 links, 74 joints
Joints:
- joint excavator_lift: limit lower=-0.1524 upper=0 effort=155.68777 velocity=0.0508 -> lower=-0.1524 upper=0 effort=311.37554 velocity=0.0508

File: src/lunabotics_model/urdf/assembly_1_sim.urdf (robot description, URDF)
Before this commit: robot assembly_1, 75 links, 74 joints
Joints:
- joint excavator_lift: limit lower=-0.1524 upper=0 effort=155.68777 velocity=0.0508 -> lower=-0.1524 upper=0 effort=311.37554 velocity=0.0508

File: src/lunabotics_model/urdf/assembly_1_sim_bekker.urdf (robot description, URDF)
Before this commit: robot assembly_1, 75 links, 74 joints
Joints:
- joint excavator_lift: limit lower=-0.1524 upper=0 effort=155.68777 velocity=0.0508 -> lower=-0.1524 upper=0 effort=311.37554 velocity=0.0508
